Commit message: nothing important for debug

File: src/rbn100_description/urdf/rbn100.xacro (robot description, xacro)
@@ -11,17 +11,15 @@
       <origin
         xyz="0 0 0"
-        rpy="0 -0.015 0" />
-      <!-- <mass
-        value="2.8925" /> -->
-      <!-- 不规则车体在仿真中滑动，增大质量 -->
+        rpy="0 0 0" />
+      <!-- 不规则车体在仿真中滑动，增大质量和比例放大惯性矩阵 -->
       <mass
-        value="30" />
+        value="29.657" />
       <inertia
-        ixx="0.066723"
-        ixy="0.00023171"
-        ixz="0.0011986"
-        iyy="0.03832"
-        iyz="-2.2372E-05"
-        izz="0.080069" />
+        ixx="0.8368808"
+        ixy="-0.0029554"
+        ixz="0.027089"
+        iyy="0.9677856"
+        iyz="0.0015188"
+        izz="1.3033017" />
     </inertial>
     <visual>
@@ -126,4 +124,284 @@
   <!-- right wheel -->
   <xacro:wheel pos="right" flag_y="-1"/>
+  <!-- 两个结构的转动惯量相对位置不均匀，导致vertical自己缓慢转动，没有转动惯量部件不会转动 -->
+  <!-- 理论上，正确的惯性矩阵加上gazebo摩擦力等的设置，就可以很稳定 -->
+  <!--
+    universal
+   -->
+  <!-- actual universal-->
+  <!-- <xacro:macro name="universal" params="pos flag_x flag_y" >
+    <link
+      name="vertical_${pos}">
+      <inertial>
+        <origin
+          xyz="0 -5.0772E-06 0.039138"
+          rpy="0 0 0" />
+        <mass
+          value="0.0095091" />
+        <inertia
+          ixx="6.8701E-06"
+          ixy="-2.7128E-10"
+          ixz="1.4028E-13"
+          iyy="6.8546E-06"
+          iyz="4.7639E-14"
+          izz="1.8597E-07" />
+      </inertial>
+      <visual>
+        <origin
+          xyz="-0.021177 0 0"
+          rpy="0 0 0" />
+        <geometry>
+          <mesh
+            filename="package://rbn100_description/meshes/vertical.dae" />
+        </geometry>
+        <material
+          name="">
+          <color
+            rgba="1 1 1 1" />
+        </material>
+      </visual>
+      <collision>
+        <origin
+          xyz="-0.021177 0 0"
+          rpy="0 0 0" />
+        <geometry>
+          <mesh
+            filename="package://rbn100_description/meshes/vertical.dae" />
+        </geometry>
+      </collision>
+    </link>
+    <joint
+      name="vertical_${pos}_joint"
+      type="continuous">
+      <origin
+        xyz="${0.15248 * flag_x} ${-0.125 * flag_y} -0.0795"
+        rpy="0 0 0" />
+      <parent
+        link="base_link" />
+      <child
+        link="vertical_${pos}" />
+      <axis
+        xyz="0 0 1" />
+    </joint>
+    <link
+      name="universal_${pos}">
+      <inertial>
+        <origin
+          xyz="4.3796E-08 -1.0791E-09 2.8229E-07"
+          rpy="0 0 0" />
+        <mass
+          value="0.075555" />
+        <inertia
+          ixx="3.1637E-05"
+          ixy="-4.9814E-11"
+          ixz="3.4396E-10"
+          iyy="6.0967E-05"
+          iyz="4.138E-11"
+          izz="3.1639E-05" />
+      </inertial>
+      <visual>
+        <origin
+          xyz="0 0 0"
+          rpy="0 0 0" />
+        <geometry>
+          <mesh
+            filename="package://rbn100_description/meshes/universal.dae" />
+        </geometry>
+        <material
+          name="">
+          <color
+            rgba="0.75686 0.73725 0.67451 1" />
+        </material>
+      </visual>
+      <collision>
+        <origin
+          xyz="0 0 0"
+          rpy="0 0 0" />
+        <geometry>
+          <mesh
+            filename="package://rbn100_description/meshes/universal.dae" />
+        </geometry>
+      </collision>
+    </link>
+    <joint
+      name="universal_${pos}_joint"
+      type="continuous">
+      <origin
+        xyz="-0.021177 0 0"
+        rpy="0 0 0" />
+      <parent
+        link="vertical_${pos}" />
+      <child
+        link="universal_${pos}" />
+      <axis
+        xyz="0 1 0" />
+    </joint>
+  </xacro:macro> -->
+  <!-- sphere universal -->
+  <xacro:macro name="universal" params="pos flag_x flag_y" >
+    <link
+      name="universal_${pos}">
+      <inertial>
+        <origin
+          xyz="0 0 0"
+          rpy="0 0 0" />
+        <mass
+          value="0.0095091" />
+        <inertia
+          ixx="5.34886875e-06"
+          ixy="0"
+          ixz="0"
+          iyy="5.34886875e-06"
+          iyz="0"
+          izz="5.34886875e-06" />
+      </inertial>
+      <visual>
+        <origin
+          xyz="0 0 0"
+          rpy="0 0 0" />
+        <geometry>
+          <sphere radius="0.0375" />
+        </geometry>
+        <material
+          name="">
+          <color
+            rgba="1 1 1 1" />
+        </material>
+      </visual>
+      <collision>
+        <origin
+          xyz="0 0 0"
+          rpy="0 0 0" />
+        <geometry>
+          <sphere radius="0.0375" />
+        </geometry>
+      </collision>
+    </link>
+    <joint
+      name="universal_${pos}_joint"
+      type="continuous">
+      <origin
+        xyz="${0.15248 * flag_x} ${-0.125 * flag_y} -0.0795"
+        rpy="0 0 0" />
+      <parent
+        link="base_link" />
+      <child
+        link="universal_${pos}" />
+      <axis
+        xyz="1 1 0" />
+    </joint>
+  </xacro:macro>
+  <xacro:universal pos="FR" flag_x="1" flag_y="1"/>
+  <xacro:universal pos="FL" flag_x="1" flag_y="-1"/>
+  <xacro:universal pos="BR" flag_x="-1" flag_y="1"/>
+  <xacro:universal pos="BL" flag_x="-1" flag_y="-1"/>
+  <!-- front caster -->
+  <link
+    name="front_caster">
+    <inertial>
+      <origin
+        xyz="-2.77555756156289E-17 -5.80442675708945E-16 0"
+        rpy="0 0 0" />
+      <mass
+        value="0.0506581815391354" />
+      <inertia
+        ixx="1.3188E-05"
+        ixy="2.1816E-22"
+        ixz="1.5232E-36"
+        iyy="1.0765E-05"
+        iyz="-1.6921E-20"
+        izz="1.3188E-05" />
+    </inertial>
+    <visual>
+      <origin
+        xyz="0 0 0"
+        rpy="0 0 0" />
+      <geometry>
+        <mesh
+          filename="package://rbn100_description/meshes/front_caster.dae" />
+      </geometry>
+      <material
+        name="">
+        <color
+          rgba="1 1 1 1" />
+      </material>
+    </visual>
+    <collision>
+      <origin
+        xyz="0 0 0"
+        rpy="0 0 0" />
+      <geometry>
+        <mesh
+          filename="package://rbn100_description/meshes/front_caster.dae" />
+      </geometry>
+    </collision>
+  </link>
+  <joint
+    name="front_caster_joint"
+    type="continuous">
+    <origin
+      xyz="0.16 0 -0.083"
+      rpy="0 0 0" />
+    <parent
+      link="base_link" />
+    <child
+      link="front_caster" />
+    <axis
+      xyz="0 1 0" />
+  </joint>
+  <!-- back caster -->
+  <link
+    name="back_caster">
+    <inertial>
+      <origin
+        xyz="2.7756E-17 -5.8981E-16 0"
+        rpy="0 0 0" />
+      <mass
+        value="0.0056549" />
+      <inertia
+        ixx="2.9759E-07"
+        ixy="-7.1138E-24"
+        ixz="-4.9678E-38"
+        iyy="4.5946E-07"
+        iyz="1.1303E-21"
+        izz="2.9759E-07" />
+    </inertial>
+    <visual>
+      <origin
+        xyz="0 0 0"
+        rpy="0 0 0" />
+      <geometry>
+        <mesh
+          filename="package://rbn100_description/meshes/back_caster.dae" />
+      </geometry>
+      <material
+        name="">
+        <color
+          rgba="1 1 1 1" />
+      </material>
+    </visual>
+    <collision>
+      <origin
+        xyz="0 0 0"
+        rpy="0 0 0" />
+      <geometry>
+        <mesh
+          filename="package://rbn100_description/meshes/back_caster.dae" />
+      </geometry>
+    </collision>
+  </link>
+  <joint
+    name="back_caster_joint"
+    type="continuous">
+    <origin
+      xyz="-0.193 0 -0.0845"
+      rpy="0 0 0" />
+    <parent
+      link="base_link" />
+    <child
+      link="back_caster" />
+    <axis
+      xyz="0 1 0" />
+  </joint>
   <!-- tof -->
   <link
@@ -464,284 +742,4 @@
   <!-- BR -->
   <xacro:cliff pos="BR" flag_x="-1" flag_y="-1"/>
-  <!-- 两个结构的转动惯量相对位置不均匀，导致vertical自己缓慢转动，没有转动惯量部件不会转动 -->
-  <!-- 理论上，正确的惯性矩阵加上gazebo摩擦力等的设置，就可以很稳定 -->
-  <!--
-    universal
-   -->
-   <!-- actual universal-->
-  <!-- <xacro:macro name="universal" params="pos flag_x flag_y" >
-    <link
-      name="vertical_${pos}">
-      <inertial>
-        <origin
-          xyz="0 -5.0772E-06 0.039138"
-          rpy="0 0 0" />
-        <mass
-          value="0.0095091" />
-        <inertia
-          ixx="6.8701E-06"
-          ixy="-2.7128E-10"
-          ixz="1.4028E-13"
-          iyy="6.8546E-06"
-          iyz="4.7639E-14"
-          izz="1.8597E-07" />
-      </inertial>
-      <visual>
-        <origin
-          xyz="-0.021177 0 0"
-          rpy="0 0 0" />
-        <geometry>
-          <mesh
-            filename="package://rbn100_description/meshes/vertical.dae" />
-        </geometry>
-        <material
-          name="">
-          <color
-            rgba="1 1 1 1" />
-        </material>
-      </visual>
-      <collision>
-        <origin
-          xyz="-0.021177 0 0"
-          rpy="0 0 0" />
-        <geometry>
-          <mesh
-            filename="package://rbn100_description/meshes/vertical.dae" />
-        </geometry>
-      </collision>
-    </link>
-    <joint
-      name="vertical_${pos}_joint"
-      type="continuous">
-      <origin
-        xyz="${0.15248 * flag_x} ${-0.125 * flag_y} -0.0795"
-        rpy="0 0 0" />
-      <parent
-        link="base_link" />
-      <child
-        link="vertical_${pos}" />
-      <axis
-        xyz="0 0 1" />
-    </joint>
-    <link
-      name="universal_${pos}">
-      <inertial>
-        <origin
-          xyz="4.3796E-08 -1.0791E-09 2.8229E-07"
-          rpy="0 0 0" />
-        <mass
-          value="0.075555" />
-        <inertia
-          ixx="3.1637E-05"
-          ixy="-4.9814E-11"
-          ixz="3.4396E-10"
-          iyy="6.0967E-05"
-          iyz="4.138E-11"
-          izz="3.1639E-05" />
-      </inertial>
-      <visual>
-        <origin
-          xyz="0 0 0"
-          rpy="0 0 0" />
-        <geometry>
-          <mesh
-            filename="package://rbn100_description/meshes/universal.dae" />
-        </geometry>
-        <material
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
Commit message: update sensor data and rates

File: src/rbn100_description/urdf/rbn100.xacro (robot description, xacro)
@@ -5,4 +5,5 @@
   <xacro:include filename="rbn100.gazebo"/>
   <link name="base_footprint"/>
+  <!-- 保持sw的参数不变，机体稳定性也会挺好，增加质量会转不动 -->
   <!-- base link -->
   <link
@@ -12,14 +13,13 @@
         xyz="0 0 0"
         rpy="0 0 0" />
-      <!-- 不规则车体在仿真中滑动，增大质量和比例放大惯性矩阵 -->
       <mass
-        value="29.657" />
+        value="2.9657" />
       <inertia
-        ixx="0.8368808"
-        ixy="-0.0029554"
-        ixz="0.027089"
-        iyy="0.9677856"
-        iyz="0.0015188"
-        izz="1.3033017" />
+        ixx="0.08368808"
+        ixy="-0.00029554"
+        ixz="0.0027089"
+        iyy="0.09677856"
+        iyz="0.00015188"
+        izz="0.13033017" />
     </inertial>
     <visual>
@@ -44,5 +44,4 @@
         <mesh
           filename="package://rbn100_description/meshes/base_link.dae" />
-        <!-- <box size="0.457 0.4 0.267" /> -->
       </geometry>
     </collision>
@@ -78,5 +77,5 @@
           ixz="1.7547E-09"
           iyy="0.0033687"
-          iyz="-3.6374E-07"
+          iyz="-3.6374E-7"
           izz="0.0019547" />
       </inertial>

Commit message: update odom data from pose to encoder

File: src/rbn100_description/urdf/rbn100.xacro (robot description, xacro)
@@ -69,8 +69,15 @@
         <origin
           xyz="-3.9818E-08 ${0.023375 * flag_y} -5.7134E-06"
-          rpy="0 0 0" />
+          rpy="-1.570796 0 0" />
         <mass
           value="1.0829" />
         <inertia
+          ixx="0.0021,"
+          ixy="0"
+          ixz="0"
+          iyy="0.0021,"
+          iyz="0"
+          izz="0.0038" />
+        <!-- <inertia
           ixx="0.0019547"
           ixy="3.8126E-10"
@@ -78,5 +85,5 @@
           iyy="0.0033687"
           iyz="-3.6374E-7"
-          izz="0.0019547" />
+          izz="0.0019547" /> -->
       </inertial>
       <visual>
@@ -96,10 +103,10 @@
       <collision>
         <origin
-          xyz="0 0 0"
-          rpy="0 0 0" />
-        <geometry>
-          <!-- <cylinder radius="0.0845" length="0.045" /> -->
-          <mesh
-            filename="package://rbn100_description/meshes/${pos}_wheel.dae" />
+          xyz="-3.9818E-08 ${0.023375 * flag_y} -5.7134E-06"
+          rpy="-1.570796 0 0" />
+        <geometry>
+          <cylinder radius="0.0845" length="0.045" />
+          <!-- <mesh
+            filename="package://rbn100_description/meshes/${pos}_wheel.dae" /> -->
         </geometry>
       </collision>
