Commit message: all modules is done except slam

File: src/rbn100_description/urdf/rbn100.xacro (robot description, xacro)
@@ -8,124 +8,68 @@
     改变碰撞属性（如主轮的）为简单形状以防止摩擦不均导致小车不走直线
    -->
-   <!-- base_footprint -->
+  <!-- base_footprint -->
   <link name="base_footprint"/>
   <!-- base link -->
-  <link
-    name="base_link">
+  <link name="base_link">
     <inertial>
-      <origin
-        xyz="0 0 0"
-        rpy="0 0 0" />
-      <mass
-        value="2.9657" />
-      <inertia
-        ixx="0.08368808"
-        ixy="-0.00029554"
-        ixz="0.0027089"
-        iyy="0.09677856"
-        iyz="0.00015188"
-        izz="0.13033017" />
+      <origin xyz="0 0 0" rpy="0 0 0" />
+      <mass value="2.9657" />
+      <inertia ixx="0.08368808" ixy="-0.00029554" ixz="0.0027089"
+                iyy="0.09677856" iyz="0.00015188"
+                izz="0.13033017" />
     </inertial>
     <visual>
-      <origin
-        xyz="0 0 0"
-        rpy="0 0 0" />
-      <geometry>
-        <mesh
-          filename="package://rbn100_description/meshes/base_link.dae" />
-      </geometry>
-      <material
-        name="">
-        <color
-          rgba="1 1 1 1" />
+      <origin xyz="0 0 0" rpy="0 0 0" />
+      <geometry>
+        <mesh filename="package://rbn100_description/meshes/base_link.dae" />
+      </geometry>
+      <material name="">
+        <color rgba="1 1 1 1" />
       </material>
     </visual>
     <collision>
-      <origin
-        xyz="0 0 0"
-        rpy="0 0 0" />
-      <geometry>
-        <mesh
-          filename="package://rbn100_description/meshes/base_link.dae" />
+      <origin xyz="0 0 0" rpy="0 0 0" />
+      <geometry>
+        <mesh filename="package://rbn100_description/meshes/base_link.dae" />
       </geometry>
     </collision>
   </link>
-  <joint
-    name="fixed"
-    type="fixed">
-    <origin
-      xyz="0 0 0.117"
-      rpy="0 0 0" />
-    <parent
-      link="base_footprint" />
-    <child
-      link="base_link" />
-    <axis
-      xyz="0 0 0" />
-  </joint>
-  <!--
-    wheel
-   -->
-   <xacro:macro name="wheel" params="pos flag_y">
-    <link
-      name="${pos}_wheel">
+  <joint name="fixed" type="fixed">
+    <origin xyz="0 0 0.117" rpy="0 0 0" />
+    <parent link="base_footprint" />
+    <child link="base_link" />
+    <axis xyz="0 0 0" />
+  </joint>
+  <!-- wheel-->
+  <xacro:macro name="wheel" params="pos flag_y">
+    <link name="${pos}_wheel">
       <inertial>
-        <origin
-          xyz="-3.9818E-08 ${0.023375 * flag_y} -5.7134E-06"
-          rpy="-1.570796 0 0" />
-        <mass
-          value="1.0829" />
-        <inertia
-          ixx="0.0021"
-          ixy="0"
-          ixz="0"
-          iyy="0.0021"
-          iyz="0"
-          izz="0.0038" />
-        <!-- <inertia
-          ixx="0.0019547"
-          ixy="3.8126E-10"
-          ixz="1.7547E-09"
-          iyy="0.0033687"
-          iyz="-3.6374E-7"
-          izz="0.0019547" /> -->
+        <origin xyz="-3.9818E-08 ${0.023375 * flag_y} -5.7134E-06" rpy="-1.570796 0 0" />
+        <mass value="1.0829" />
+        <inertia ixx="0.0021" ixy="0" ixz="0"
+                 iyy="0.0021" iyz="0"
+                 izz="0.0038" />
       </inertial>
       <visual>
-        <origin
-          xyz="0 0 0"
-          rpy="0 0 0" />
-        <geometry>
-          <mesh
-            filename="package://rbn100_description/meshes/${pos}_wheel.dae" />
-        </geometry>
-        <material
-          name="">
-          <color
-            rgba="0.2 0.2 0.2 1" />
+        <origin xyz="0 0 0" rpy="0 0 0" />
+        <geometry>
+          <mesh filename="package://rbn100_description/meshes/${pos}_wheel.dae" />
+        </geometry>
+        <material name="">
+          <color rgba="0.2 0.2 0.2 1" />
         </material>
       </visual>
       <collision>
-        <origin
-          xyz="-3.9818E-08 ${0.023375 * flag_y} -5.7134E-06"
-          rpy="-1.570796 0 0" />
+        <origin xyz="-3.9818E-08 ${0.023375 * flag_y} -5.7134E-06" rpy="-1.570796 0 0" />
         <geometry>
           <cylinder radius="0.0845" length="0.045" />
-          <!-- <mesh
-            filename="package://rbn100_description/meshes/${pos}_wheel.dae" /> -->
         </geometry>
       </collision>
     </link>
-    <joint
-      name="${pos}_wheel_joint"
-      type="continuous">
-      <origin
-        xyz="0 ${0.13755 * flag_y} -0.0325"
-        rpy="0 0 0" />
-      <parent
-        link="base_link" />
-      <child
-        link="${pos}_wheel" />
-      <axis
-        xyz="0 1 0" />
+    <joint name="${pos}_wheel_joint" type="continuous">
+      <origin xyz="0 ${0.13755 * flag_y} -0.0325" rpy="0 0 0" />
+      <parent link="base_link" />
+      <child link="${pos}_wheel" />
+      <axis xyz="0 1 0" />
     </joint>
   </xacro:macro>
@@ -135,5 +79,4 @@
   <xacro:wheel pos="right" flag_y="-1"/>
   <!-- 两个结构的转动惯量相对位置不均匀，导致vertical自己缓慢转动，没有转动惯量部件不会转动 -->
-  <!-- 理论上，正确的惯性矩阵加上gazebo摩擦力等的设置，就可以很稳定 -->
   <!--
     universal
@@ -141,146 +84,90 @@
   <!-- actual universal-->
   <!-- <xacro:macro name="universal" params="pos flag_x flag_y" >
-    <link
-      name="vertical_${pos}">
+    <link name="vertical_${pos}">
       <inertial>
-        <origin
-          xyz="0 -5.0772E-06 0.039138"
-          rpy="0 0 0" />
-        <mass
-          value="0.0095091" />
-        <inertia
-          ixx="6.8701E-06"
-          ixy="-2.7128E-10"
-          ixz="1.4028E-13"
-          iyy="6.8546E-06"
-          iyz="4.7639E-14"
-          izz="1.8597E-07" />
+        <origin xyz="0 -5.0772E-06 0.039138" rpy="0 0 0" />
+        <mass value="0.0095091" />
+        <inertia ixx="6.8701E-06" ixy="-2.7128E-10" ixz="1.4028E-13"
+                 iyy="6.8546E-06" iyz="4.7639E-14"
+                 izz="1.8597E-07" />
       </inertial>
       <visual>
-        <origin
-          xyz="-0.021177 0 0"
-          rpy="0 0 0" />
-        <geometry>
-          <mesh
-            filename="package://rbn100_description/meshes/vertical.dae" />
-        </geometry>
-        <material
-          name="">
-          <color
-            rgba="1 1 1 1" />
+        <origin xyz="-0.021177 0 0" rpy="0 0 0" />
+        <geometry>
+          <mesh filename="package://rbn100_description/meshes/vertical.dae" />
+        </geometry>
+        <material name="">
+          <color rgba="1 1 1 1" />
         </material>
       </visual>
       <collision>
-        <origin
-          xyz="-0.021177 0 0"
-          rpy="0 0 0" />
-        <geometry>
-          <mesh
-            filename="package://rbn100_description/meshes/vertical.dae" />
+        <origin xyz="-0.021177 0 0" rpy="0 0 0" />
+        <geometry>
+          <mesh filename="package://rbn100_description/meshes/vertical.dae" />
         </geometry>
       </collision>
     </link>
-    <joint
-      name="vertical_${pos}_joint"
-      type="continuous">
-      <origin
-        xyz="${0.15248 * flag_x} ${-0.125 * flag_y} -0.0795"
-        rpy="0 0 0" />
-      <parent
-        link="base_link" />
-      <child
-        link="vertical_${pos}" />
-      <axis
-        xyz="0 0 1" />
-    </joint>
-    <link
-      name="universal_${pos}">
+    <joint name="vertical_${pos}_joint" type="continuous">
+      <origin xyz="${0.15248 * flag_x} ${-0.125 * flag_y} -0.0795" rpy="0 0 0" />
+      <parent link="base_link" />
+      <child link="vertical_${pos}" />
+      <axis xyz="0 0 1" />
+    </joint>
+    <link name="universal_${pos}">
       <inertial>
-        <origin
-          xyz="4.3796E-08 -1.0791E-09 2.8229E-07"
-          rpy="0 0 0" />
-        <mass
-          value="0.075555" />
-        <inertia
-          ixx="3.1637E-05"
-          ixy="-4.9814E-11"
-          ixz="3.4396E-10"
-          iyy="6.0967E-05"
-          iyz="4.138E-11"
-          izz="3.1639E-05" />
+        <origin xyz="4.3796E-08 -1.0791E-09 2.8229E-07" rpy="0 0 0" />
+        <mass value="0.075555" />
+        <inertia ixx="3.1637E-05" ixy="-4.9814E-11" ixz="3.4396E-10"
+                 iyy="6.0967E-05" iyz="4.138E-11"
+                 izz="3.1639E-05" />
       </inertial>
       <visual>
-        <origin
-          xyz="0 0 0"
-          rpy="0 0 0" />
-        <geometry>
-          <mesh
-            filename="package://rbn100_description/meshes/universal.dae" />
-        </geometry>
-        <material
-          name="">
-          <color
-            rgba="0.75686 0.73725 0.67451 1" />
+        <origin xyz="0 0 0" rpy="0 0 0" />
+        <geometry>
+          <mesh filename="package://rbn100_description/meshes/universal.dae" />
+        </geometry>
+        <material name="">
+          <color rgba="0.75686 0.73725 0.67451 1" />
         </material>
       </visual>
       <collision>
-        <origin
-          xyz="0 0 0"
-          rpy="0 0 0" />
-        <geometry>
-          <mesh
-            filename="package://rbn100_description/meshes/universal.dae" />
+        <origin xyz="0 0 0" rpy="0 0 0" />
+        <geometry>
+          <mesh filename="package://rbn100_description/meshes/universal.dae" />
         </geometry>
       </collision>
     </link>
-    <joint
-      name="universal_${pos}_joint"
-      type="continuous">
-      <origin
-        xyz="-0.021177 0 0"
-        rpy="0 0 0" />
-      <parent
-        link="vertical_${pos}" />
-      <child
-        link="universal_${pos}" />
-      <axis
-        xyz="0 1 0" />
+    <joint name="universal_${pos}_joint" type="continuous">
+      <origin xyz="-0.021177 0 0"  rpy="0 0 0" />
+      <parent link="vertical_${pos}" />
+      <child link="universal_${pos}" />
+      <axis xyz="0 1 0" />
     </joint>
   </xacro:macro> -->
   <!-- sphere universal -->
+  <!--
+    fixed joint with very small friction for vehicle to stand right still,
+    and have very small effect on vehicle's move.
+   -->
   <xacro:macro name="universal" params="pos flag_x flag_y" >
-    <link
-      name="universal_${pos}">
+    <link name="universal_${pos}">
       <inertial>
-        <origin
-          xyz="0 0 0"
-          rpy="0 0 0" />
-        <mass
-          value="0.0095091" />
-        <inertia
-          ixx="5.34886875e-06"
-          ixy="0"
-          ixz="0"
-          iyy="5.34886875e-06"
-          iyz="0"
-          izz="5.34886875e-06" />
+        <origin xyz="0 0 0" rpy="0 0 0" />
+        <mass value="0.0095091" />
+        <inertia ixx="5.34886875e-06" ixy="0" ixz="0"
+                 iyy="5.34886875e-06" iyz="0"
+                 izz="5.34886875e-06" />
       </inertial>
       <visual>
-        <origin
-          xyz="0 0 0"
-          rpy="0 0 0" />
+        <origin xyz="0 0 0" rpy="0 0 0" />
         <geometry>
           <sphere radius="0.0375" />
         </geometry>
-        <material
-          name="">
-          <color
-            rgba="1 1 1 1" />
+        <material name="">
+          <color rgba="1 1 1 1" />
         </material>
       </visual>
       <collision>
-        <origin
-          xyz="0 0 0"
-          rpy="0 0 0" />
+        <origin xyz="0 0 0" rpy="0 0 0" />
         <geometry>
           <sphere radius="0.0375" />
@@ -288,16 +175,8 @@
       </collision>
     </link>
-    <joint
-      name="universal_${pos}_joint"
-      type="continuous">
-      <origin
-        xyz="${0.15248 * flag_x} ${-0.125 * flag_y} -0.0795"
-        rpy="0 0 0" />
-      <parent
-        link="base_link" />
-      <child
-        link="universal_${pos}" />
-      <axis
-        xyz="1 1 0" />
+    <joint name="universal_${pos}_joint" type="fixed">
+      <origin xyz="${0.15248 * flag_x} ${-0.125 * flag_y} -0.0795" rpy="0 0 0" />
+      <parent link="base_link" />
+      <child link="universal_${pos}" />
     </joint>
   </xacro:macro>
@@ -307,281 +186,143 @@
   <xacro:universal pos="BL" flag_x="-1" flag_y="-1"/>
   <!-- front caster -->
-  <link
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
Commit message: carding procedure of gazebo model plugin

File: src/rbn100_description/urdf/rbn100.xacro (robot description, xacro)
@@ -3,12 +3,5 @@
   <xacro:include filename="materials.xacro"/>
   <xacro:include filename="rbn100.gazebo"/>
-  <!--
-    urdf：ros中机器描述格式，在rviz中显示，gazebo会转换为sdf再显示；
-    一般保持sw的参数不变，增加质量小车可能会转不动;
-    改变碰撞属性（如主轮的）为简单形状以防止摩擦不均导致小车不走直线
-   -->
-  <!-- base_footprint -->
   <link name="base_footprint"/>
-  <!-- base link -->
   <link name="base_link">
     <inertial>
@@ -74,7 +67,5 @@
     </joint>
   </xacro:macro>
-  <!-- left wheel -->
   <xacro:wheel pos="left" flag_y="1"/>
-  <!-- right wheel -->
   <xacro:wheel pos="right" flag_y="-1"/>
   <!-- 两个结构的转动惯量相对位置不均匀，导致vertical自己缓慢转动，没有转动惯量部件不会转动 -->
@@ -284,5 +275,4 @@
   <!-- camera -->
   <xacro:macro name="camera" params="name pos">
-    <!-- body -->
     <joint name="fisheye_${name}_joint" type="fixed">
       <origin xyz="0 ${pos * 0.035} 0" rpy="0 0 0" />
@@ -291,5 +281,4 @@
     </joint>
     <link name="fisheye_${name}_frame" />
-    <!-- optical -->
     <joint name="fisheye_${name}_optical_joint" type="fixed">
       <origin xyz="0.02 0 0" rpy="0 0 0" />
@@ -328,55 +317,57 @@
   <!--
     sonar
-   -->
-   <xacro:macro name="sonar" params="pos">
-    <link name="sonar_${pos}">
-      <visual>
-        <origin xyz="0 0 0" rpy="0 0 0" />
-        <geometry>
-          <box size="0.0015 0.05 0.02"/>
-        </geometry>
-        <material name="">
-          <color rgba="0 0 0 1" />
-        </material>
-      </visual>
-    </link>
-   </xacro:macro>
-   <!-- back -->
-  <xacro:sonar pos="back"/>
+  -->
+  <xacro:macro name="sonar" params="pos">
+  <link name="sonar_${pos}_link">
+    <visual>
+      <origin xyz="0 0 0" rpy="0 0 0" />
+      <geometry>
+        <box size="0.0015 0.05 0.02"/>
+      </geometry>
+      <material name="">
+        <color rgba="0 0 0 1" />
+      </material>
+    </visual>
+  </link>
+  </xacro:macro>
   <joint name="back_sonar_joint" type="fixed">
     <origin xyz="-0.233 0 0.063" rpy="0 0 3.14" />
     <parent link="base_link" />
-    <child link="sonar_back" />
-    <axis xyz="0 0 0" />
-  </joint>
-  <!-- front -->
-  <xacro:sonar pos="front"/>
+    <child link="sonar_back_link" />
+    <axis xyz="0 0 0" />
+  </joint>
+  <xacro:sonar pos="back"/>
   <joint name="front_sonar_joint" type="fixed">
     <origin xyz="0.2316 0 0.063" rpy="0 0 0" />
     <parent link="base_link" />
-    <child link="sonar_front" />
-    <axis xyz="0 0 0" />
-  </joint>
-  <!-- FL -->
-  <xacro:sonar pos="FL"/>
+    <child link="sonar_front_link" />
+    <axis xyz="0 0 0" />
+  </joint>
+  <xacro:sonar pos="front"/>
   <joint name="sonar_FL_joint" type="fixed">
     <origin xyz="0.21648 0.17249 0.063" rpy="0 0 0.628" />
     <parent link="base_link" />
-    <child link="sonar_FL" />
-    <axis xyz="0 0 0" />
-  </joint>
-  <!-- FR -->
-  <xacro:sonar pos="FR"/>
+    <child link="sonar_FL_link" />
+    <axis xyz="0 0 0" />
+  </joint>
+  <xacro:sonar pos="FL"/>
   <joint name="sonar_FR_joint" type="fixed">
     <origin xyz="0.21748 -0.17249 0.063" rpy="0 0 -0.628" />
     <parent link="base_link" />
-    <child link="sonar_FR" />
-    <axis xyz="0 0 0" />
-  </joint>
+    <child link="sonar_FR_link" />
+    <axis xyz="0 0 0" />
+  </joint>
+  <xacro:sonar pos="FR"/>
   <!--
     cliff
    -->
   <xacro:macro name="cliff" params="pos flag_x flag_y" >
-    <link name="cliff_${pos}">
+    <joint name="cliff_${pos}_joint" type="fixed">
+      <origin xyz="${0.106 * flag_x} ${0.1865 * flag_y} -0.0609" rpy="0 1.570796 0" />
+      <parent link="base_link" />
+      <child link="cliff_${pos}_link" />
+      <axis xyz="0 0 0" />
+    </joint>
+    <link name="cliff_${pos}_link">
       <visual>
         <origin xyz="0 0 0" rpy="0 0 0" />
@@ -389,20 +380,16 @@
       </visual>
     </link>
-    <joint name="cliff_${pos}_joint" type="fixed">
-      <origin xyz="${0.106 * flag_x} ${0.1865 * flag_y} -0.0609" rpy="0 1.570796 0" />
-      <parent link="base_link" />
-      <child link="cliff_${pos}" />
-      <axis xyz="0 0 0" />
-    </joint>
   </xacro:macro>
-  <!-- FL -->
   <xacro:cliff pos="FL" flag_x="1" flag_y="1"/>
-  <!-- FR -->
   <xacro:cliff pos="FR" flag_x="1" flag_y="-1"/>
-  <!-- BL -->
   <xacro:cliff pos="BL" flag_x="-1" flag_y="1"/>
-  <!-- BR -->
   <xacro:cliff pos="BR" flag_x="-1" flag_y="-1"/>
   <!-- bumper -->
+  <joint name="bumper_joint" type="fixed">
+    <origin xyz="0.1115 0.001 -0.077" rpy="0 0 0" />
+    <parent link="base_link" />
+    <child link="bumper" />
+    <axis xyz="0 0 0" />
+  </joint>
   <link name="bumper">
     <inertial>
@@ -429,10 +416,4 @@
     </collision>
   </link>
-  <joint name="bumper_joint" type="fixed">
-    <origin xyz="0.1115 0.001 -0.077" rpy="0 0 0" />
-    <parent link="base_link" />
-    <child link="bumper" />
-    <axis xyz="0 0 0" />
-  </joint>
   <!-- transmission, parsed by ros_control -->
   <!-- <transmission name="left_wheel_joint_trans">
